File: Technische Zeichnungen/Eagle/Pfeffer_Ribbon/pfeffer_main_circuit.sch (EAGLE design)
At the start: 12 parts

Commit message: added ribbon testing, firmware and applied it to the new firmware, added a new tech. drawing, added new PCB layouts
Parts:
- R11: value 100k -> 24
Connections:
- net N$10: now also MC_RIGHT.7, RIBBON_CONNECTOR.3; no longer MC_RIGHT.6, RIBBON_CONNECTOR.2
- net N$11: now also R5.2; no longer RIBBON_CONNECTOR.3
- net N$9: now also MC_RIGHT.6, RIBBON_CONNECTOR.2; no longer MC_RIGHT.7, R5.2
Other:
- moved on the sheet: R5, RIBBON_CONNECTOR
Changed lines of the file:
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@@
 <part name="MAIN2SUB" library="pinhead" deviceset="PINHD-1X4" device=""/>
 <part name="GND6" library="supply1" deviceset="GND" device=""/>
-<part name="R11" library="rcl" deviceset="R-EU_" device="0204/7" value="100k"/>
+<part name="R11" library="rcl" deviceset="R-EU_" device="0204/7" value="24"/>
 <part name="GND10" library="supply1" deviceset="GND" device="" value="GND"/>
 <part name="P+2" library="supply1" deviceset="VCC" device="" value="3.3V"/>
@@
 <instance part="U$1" gate="2" x="101.6" y="7.62"/>
 <instance part="GND11" gate="1" x="91.44" y="12.7" rot="R270"/>
-<instance part="RIBBON_CONNECTOR" gate="A" x="104.14" y="25.4"/>
-<instance part="R5" gate="G$1" x="78.74" y="22.86" rot="MR0"/>
+<instance part="RIBBON_CONNECTOR" gate="A" x="30.48" y="81.28" rot="R270"/>
+<instance part="R5" gate="G$1" x="48.26" y="20.32" rot="MR180"/>
 </instances>
 <busses>
@@
 </segment>
 </net>
-<net name="N$7" class="0">
-<segment>
-<pinref part="MC_RIGHT" gate="G$1" pin="5"/>
-<pinref part="RIBBON_CONNECTOR" gate="A" pin="1"/>
-<wire x1="63.5" y1="27.94" x2="101.6" y2="27.94" width="0.1524" layer="91"/>
-</segment>
-</net>
-<net name="N$10" class="0">
-<segment>
-<pinref part="RIBBON_CONNECTOR" gate="A" pin="2"/>
-<pinref part="MC_RIGHT" gate="G$1" pin="6"/>
-<wire x1="63.5" y1="25.4" x2="86.36" y2="25.4" width="0.1524" layer="91"/>
-<pinref part="R5" gate="G$1" pin="1"/>
-<wire x1="86.36" y1="25.4" x2="101.6" y2="25.4" width="0.1524" layer="91"/>
-<wire x1="83.82" y1="22.86" x2="86.36" y2="22.86" width="0.1524" layer="91"/>
-<wire x1="86.36" y1="22.86" x2="86.36" y2="25.4" width="0.1524" layer="91"/>
-<junction x="86.36" y="25.4"/>
-</segment>
-</net>
-<net name="N$11" class="0">
-<segment>
-<pinref part="MC_RIGHT" gate="G$1" pin="8"/>
-<wire x1="63.5" y1="20.32" x2="88.9" y2="20.32" width="0.1524" layer="91"/>
-<wire x1="88.9" y1="20.32" x2="88.9" y2="22.86" width="0.1524" layer="91"/>
-<pinref part="RIBBON_CONNECTOR" gate="A" pin="3"/>
-<wire x1="88.9" y1="22.86" x2="101.6" y2="22.86" width="0.1524" layer="91"/>
-</segment>
-</net>
 <net name="N$5" class="0">
 <segment>
@@
 </segment>
 </net>
+<net name="N$7" class="0">
+<segment>
+<pinref part="RIBBON_CONNECTOR" gate="A" pin="1"/>
+<wire x1="33.02" y1="83.82" x2="33.02" y2="60.96" width="0.1524" layer="91"/>
+<wire x1="33.02" y1="60.96" x2="53.34" y2="60.96" width="0.1524" layer="91"/>
+<wire x1="53.34" y1="60.96" x2="53.34" y2="27.94" width="0.1524" layer="91"/>
+<pinref part="MC_RIGHT" gate="G$1" pin="5"/>
+<wire x1="53.34" y1="27.94" x2="63.5" y2="27.94" width="0.1524" layer="91"/>
+</segment>
+</net>
 <net name="N$9" class="0">
 <segment>
+<pinref part="RIBBON_CONNECTOR" gate="A" pin="2"/>
+<wire x1="30.48" y1="83.82" x2="30.48" y2="58.42" width="0.1524" layer="91"/>
+<wire x1="30.48" y1="58.42" x2="50.8" y2="58.42" width="0.1524" layer="91"/>
+<wire x1="50.8" y1="58.42" x2="50.8" y2="25.4" width="0.1524" layer="91"/>
+<pinref part="MC_RIGHT" gate="G$1" pin="6"/>
+<wire x1="50.8" y1="25.4" x2="63.5" y2="25.4" width="0.1524" layer="91"/>
+</segment>
+</net>
+<net name="N$10" class="0">
+<segment>
+<pinref part="RIBBON_CONNECTOR" gate="A" pin="3"/>
+<wire x1="27.94" y1="83.82" x2="27.94" y2="55.88" width="0.1524" layer="91"/>
+<wire x1="27.94" y1="55.88" x2="43.18" y2="55.88" width="0.1524" layer="91"/>
+<wire x1="43.18" y1="55.88" x2="43.18" y2="22.86" width="0.1524" layer="91"/>
 <pinref part="MC_RIGHT" gate="G$1" pin="7"/>
+<wire x1="43.18" y1="22.86" x2="63.5" y2="22.86" width="0.1524" layer="91"/>
+<pinref part="R5" gate="G$1" pin="1"/>
+<wire x1="43.18" y1="22.86" x2="43.18" y2="20.32" width="0.1524" layer="91"/>
+<junction x="43.18" y="22.86"/>
+</segment>
+</net>
+<net name="N$11" class="0">
+<segment>
 <pinref part="R5" gate="G$1" pin="2"/>
-<wire x1="63.5" y1="22.86" x2="73.66" y2="22.86" width="0.1524" layer="91"/>
-</segment>
-</net>
+<pinref part="MC_RIGHT" gate="G$1" pin="8"/>
+<wire x1="53.34" y1="20.32" x2="63.5" y2="20.32" width="0.1524" layer="91"/>
+</segment>
+</net>
